Commit message: update

File: src/rover_description/urdf/simple_4wd_rover_sameid_2bus.urdf.xacro (robot description, xacro)
@@ -4,12 +4,14 @@
   <xacro:arg name="can_left"  default="can0"/>
   <xacro:arg name="can_right" default="can1"/>
-  <!-- Geometry -->
-  <xacro:arg name="wheel_radius" default="0.10"/>
-  <xacro:arg name="wheel_width"  default="0.05"/>
-  <xacro:arg name="track_width"  default="0.50"/>
-  <xacro:arg name="wheelbase"    default="0.60"/>
-  <xacro:arg name="chassis_length" default="0.65"/>
-  <xacro:arg name="chassis_width"  default="0.45"/>
-  <xacro:arg name="chassis_height" default="0.12"/>
+  <xacro:property name="can_left"  value="$(arg can_left)"/>
+  <xacro:property name="can_right" value="$(arg can_right)"/>
+  <!-- Geometry (hardcoded) -->
+  <xacro:property name="wheel_radius"   value="0.10"/>
+  <xacro:property name="wheel_width"    value="0.05"/>
+  <xacro:property name="track_width"    value="0.50"/>
+  <xacro:property name="wheelbase"      value="0.60"/>
+  <xacro:property name="chassis_length" value="0.65"/>
+  <xacro:property name="chassis_width"  value="0.45"/>
+  <xacro:property name="chassis_height" value="0.12"/>
   <!-- AK45-36 constants -->
   <xacro:property name="pole_pairs" value="14"/>
