Commit message: update

File: src/rover_description/urdf/four_wheel.urdf.xacro (robot description, xacro)
@@ -4,7 +4,7 @@
   <xacro:arg name="can_interface" default="can0"/>
   <!-- Geometry -->
-  <xacro:arg name="wheel_radius" default="0.10"/>
+  <xacro:arg name="wheel_radius" default="0.1016"/>
   <xacro:arg name="wheel_width"  default="0.05"/>
-  <xacro:arg name="track_width"  default="0.50"/>  <!-- center-to-center left-right -->
+  <xacro:arg name="track_width"  default="0.6858"/>  <!-- center-to-center left-right (27 in) -->
   <xacro:arg name="wheelbase"    default="0.60"/>  <!-- center-to-center front-rear -->
   <xacro:arg name="chassis_length" default="0.65"/>

File: src/rover_description/urdf/one_wheel.urdf.xacro (robot description, xacro)
@@ -3,5 +3,5 @@
   <!-- Parameters you can override from launch -->
   <xacro:arg name="can_interface" default="can0"/>
-  <xacro:arg name="wheel_radius" default="0.10"/>
+  <xacro:arg name="wheel_radius" default="0.1016"/>
   <xacro:arg name="wheel_width"  default="0.05"/>
   <!-- AK45-36 constants (override if you swap actuator model) -->

File: src/rover_description/urdf/simple_4wd_rover_sameid_2bus.urdf.xacro (robot description, xacro)
@@ -7,7 +7,7 @@
   <xacro:property name="can_right" value="$(arg can_right)"/>
   <!-- Geometry (hardcoded) -->
-  <xacro:property name="wheel_radius"   value="0.10"/>
+  <xacro:property name="wheel_radius"   value="0.1016"/>
   <xacro:property name="wheel_width"    value="0.05"/>
-  <xacro:property name="track_width"    value="0.50"/>
+  <xacro:property name="track_width"    value="0.6858"/>
   <xacro:property name="wheelbase"      value="0.60"/>
   <xacro:property name="chassis_length" value="0.65"/>
